File: pcb/throwing_bagels.brd (EAGLE design)
At the start: 165.1 x 165.1 mm, 41 parts

Commit message: Demo board v1.0.0
Parts:
- removed C2: (no value), throwing_bagels:ADAFRUIT_E2,5-6E
- added LED1, LED2, LED3, LED4: (no value), adafruit:CHIPLED_0603
- added R1, R2, R3, R4: (no value), SparkFun-Resistors:0603
- moved XT5 69.9 mm to (-38.1, 29.2), turned to 0 degrees
- moved JP1 64.8 mm to (-33.0, 22.9)
- moved C1 9.92 mm to (-38.1, 24.1), turned to 180 degrees
- moved BBB 0.57 mm to (27.9, 44.5)
Connections:
- new net N$1: LED4.C, R4.1
- new net N$10: LED3.C, R3.1
- new net N$11: LED2.C, R2.1
- new net N$17: LED1.C, R1.1
- net 5V_1: now also LED1.A
- net 5V_2: now also JP1.1, LED2.A
- net 5V_3: now also LED3.A
- net 5V_4: now also LED4.A; no longer JP1.1
- net 5V_BBB: no longer C2.+
- net GND: now also R1.2, R2.2, R3.2, R4.2; no longer C2.-
Routing:
- net S17: track 0.00 -> 126.9 mm, vias 0 -> 3
- net S31: track 0.00 -> 122.5 mm, vias 0 -> 1
- net S12: track 0.00 -> 111.7 mm, vias 0 -> 1
- net S29: track 0.00 -> 110.6 mm, vias 0 -> 2
- net S30: track 0.00 -> 109.0 mm, vias 0 -> 3
- net S11: track 0.00 -> 103.1 mm, vias 0 -> 1
- net S10: track 0.00 -> 101.8 mm, vias 0 -> 2
- net S28: track 0.00 -> 99.2 mm, vias 0 -> 3
- net S27: track 0.00 -> 96.5 mm, vias 0 -> 2
- net S26: track 0.00 -> 96.2 mm, vias 0 -> 2
- net S21: track 0.00 -> 94.3 mm, vias 0 -> 1
- net S25: track 0.00 -> 88.7 mm, vias 0 -> 3
- net S24: track 0.00 -> 86.4 mm, vias 0 -> 2
- net S9: track 0.00 -> 85.7 mm, vias 0 -> 2
- net S22: track 0.00 -> 81.7 mm, vias 0 -> 1
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- added copper zone on layer 1, net 5V_BBB
Other:
- outline, holes or cut-outs redrawn
- board text added: "5V ONLY"
- board text added: "5V_1"
- board text added: "5V_1 PWR"
- board text added: "5V_2"
- board text added: "5V_2 PWR"
- board text added: "5V_3"
- board text added: "5V_3 PWR"
- board text added: "5V_4"
- board text added: "5V_4 PWR"
- board text added: "5V_BBB"
- board text added: "BBB_PWR"
- board text added: "ThrowingBagels Demo Board"
- board text added: "v1.0.0 - jp@iontank.com 2020"
