File: pcb/throwing_bagels.sch (EAGLE design)
At the start: 41 parts

Commit message: Demo board v1.0.0
Parts:
- removed C2: (no value), throwing_bagels:ADAFRUIT_CPOL-USE2,5-6E
- added LED1, LED2, LED3, LED4: (no value), adafruit:LEDCHIPLED_0603
- added R1, R2, R3, R4: (no value), SparkFun-Resistors:RESISTOR0603
Connections:
- new net N$1: LED4.C, R4.1
- new net N$10: LED3.C, R3.1
- new net N$11: LED2.C, R2.1
- new net N$17: LED1.C, R1.1
- net 5V_1: now also LED1.A
- net 5V_2: now also JP1.1, LED2.A
- net 5V_3: now also LED3.A
- net 5V_4: now also LED4.A; no longer JP1.1
- net 5V_BBB: no longer C2.+
- net GND: now also R1.2, R2.2, R3.2, R4.2; no longer C2.-
Other:
- moved on the sheet: JP1
